File: MCU_Pins_Sockets.kicad_sch (KiCad schematic)
At the start: 5 parts, among them J1 Conn_01x15_Pin, J2 Conn_01x15_Socket, J3 Conn_01x15_Pin, J4 Conn_01x15_Socket

Commit message: peripheral changes
Signed-off-by: deyviaa <legoked@gmail.com>
Connections:
- new net A0: A1.19 (A0), J1.4 (Pin_4), J2.4 (Pin_4)
- new net B0: A1.18 (B0), J1.3 (Pin_3), J2.3 (Pin_3)
- new net VIN: A1.30 (VIN), J1.15 (Pin_15), J2.15 (Pin_15)
