File: ArdNanoESP32_DevBoard.kicad_pcb (KiCad board)
At the start: 2 copper layers, 163 x 77.6 mm, 48 parts, among them J1 Conn_01x15_Pin, J2 Conn_01x15_Socket, J3 Conn_01x15_Pin, J4 Conn_01x15_Socket, J5 Conn_01x04, J6 Conn_01x04, J7 Conn_01x04, J8 Conn_01x05, K1 SW_Push, K2 SW_Push, K3 SW_Push, K4 SW_Push, SW1 SW_SPDT, SW2 SW_SPDT, SW3 SW_SPDT, SW4 SW_SPDT, SW9 SW_SPDT

Commit message: the rest lol
Signed-off-by: deyviaa <legoked@gmail.com>
Parts:
- moved +3V3 100.7 mm to (151.0, 97.5), turned to -90 degrees
- moved C1 78.5 mm to (46.5, 28.6), turned to 0 degrees
- moved D1 77.1 mm to (41.5, 31.1), turned to -90 degrees
- moved R15 75.0 mm to (130.6, 37.0), turned to 0 degrees
- moved R14 74.5 mm to (130.6, 38.5), turned to 0 degrees
- moved GND 67.4 mm to (101.8, 30.1), turned to -90 degrees
- moved R5 66.5 mm to (46.5, 33.5), turned to 180 degrees
- moved I2C1 65.3 mm to (129.2, 32.9), turned to 180 degrees
- moved LED4 47.4 mm to (66.1, 31.1), turned to 90 degrees
- moved LED3 46.5 mm to (61.7, 31.1), turned to 90 degrees
- moved LED2 45.4 mm to (57.4, 31.1), turned to 90 degrees
- moved LED1 43.9 mm to (53.1, 31.1), turned to 90 degrees
- moved R4 42.4 mm to (67.0, 28.6)
- moved R3 41.3 mm to (62.6, 28.6)
- moved R2 40.1 mm to (58.3, 28.6)
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- renumbered J6 to +3V3, J5 to +5V, REF**2 to ?, REF**3 to ?, REF**1 to ?, J7 to GND, D2 to LED1, D3 to LED2, D4 to LED3, D5 to LED4
Connections:
- net Net-(BZ1-+) renamed /Peripherals/BUZZ_ANODE
- net Net-(D1-DIN) renamed /Peripherals/RGB_ANODE
- net Net-(D2-A) renamed /Peripherals/LED1_ANODE
- net Net-(D3-A) renamed /Peripherals/LED2_ANODE
- net Net-(D4-A) renamed /Peripherals/LED3_ANODE
- net Net-(D5-A) renamed /Peripherals/LED4_ANODE
- net Net-(J1-Pin_15) renamed /MCU_Pins_Sockets/VIN
- net Net-(J1-Pin_3) renamed /MCU_Pins_Sockets/B0
- net Net-(J1-Pin_4) renamed /MCU_Pins_Sockets/A0
- net Net-(SW1-B) renamed /Peripherals/SW1_COM
- net Net-(SW2-B) renamed /Peripherals/SW2_COM
- net Net-(SW3-B) renamed /Peripherals/SW3_COM
- net Net-(SW4-B) renamed /Peripherals/SW4_COM
- net Net-(SW9-B) renamed /Peripherals/SW9_COM
Routing:
- net 3V3: track 0.00 -> 235.4 mm, vias 0 -> 4
- net VUSB: track 0.00 -> 147.3 mm, vias 0 -> 4
- net /Peripherals/BUZZ: track 0.00 -> 94.8 mm
- net /Peripherals/K1: track 0.00 -> 60.5 mm
- net /Peripherals/POT: track 0.00 -> 54.3 mm
- net A5: track 0.00 -> 50.9 mm
- net A4: track 0.00 -> 48.0 mm
- net /Peripherals/K2: track 0.00 -> 47.2 mm
- net /Peripherals/LED1: track 0.00 -> 35.5 mm
- net /Peripherals/K3: track 0.00 -> 34.0 mm
- net /Peripherals/RGB: track 0.00 -> 32.3 mm
- net /Peripherals/LED2: track 0.00 -> 28.2 mm
- net /Peripherals/SW3_COM: track 0.00 -> 27.9 mm
- net /Peripherals/SW4_COM: track 0.00 -> 23.6 mm, vias 0 -> 2
- net /Peripherals/LED3: track 0.00 -> 21.0 mm
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Other:
- board text added: "3V3"
- board text added: "A0"
- board text added: "A1"
- board text added: "A2"
- board text added: "A3"
- board text added: "A4"
- board text added: "A5"
- board text added: "A6"
- board text added: "A7"
- board text added: "B0"
- board text added: "B1"
- board text added: "BUZZ"
- board text added: "D1/TX"
- board text added: "D10"
- board text added: "D11"
- board text added: "D12"
- board text added: "D13"
- board text added: "D2"
- board text added: "D3"
- board text added: "D4"
- board text added: "D5"
- board text added: "D6"
- board text added: "D7"
- board text added: "D8"
- board text added: "D9"
- board text added: "K1"
- board text added: "K2"
- board text added: "K3"
- board text added: "K4"
- board text added: "LED1"
- board text added: "LED2"
- board text added: "LED3"
- board text added: "LED4"
- board text added: "POT"
- board text added: "RGB"
- board text added: "RST"
- board text added: "RX0"
- board text added: "SW1"
- board text added: "SW2"
- board text added: "SW3"
- board text added: "SW4"
- board text added: "VIN"
- board text added: "VUSB"
